File: Kicad/EDMX/EDMX.kicad_sch (KiCad schematic)
At the start: 14 parts, among them J1 XLR3 IN, J2 Conn_01x04, J3 XLR3 OUT, Q1 2N3904, U1 MAX485E, U2 XIAO-ESP32-C3-DIP

Commit message: nano
Parts:
- added D4: DMX Status, LED_SMD:LED_WS2812B_PLCC4_5.0x5.0mm_P3.2mm, symbol LED:WS2812B
- added D5: WiFi Status, LED_SMD:LED_WS2812B_PLCC4_5.0x5.0mm_P3.2mm, symbol LED:WS2812B
- added D6: Light Control, LED_SMD:LED_WS2812B_PLCC4_5.0x5.0mm_P3.2mm, symbol LED:WS2812B
Connections:
- net GND: now also D4.3 (VSS), D5.3 (VSS), D6.3 (VSS)
- net +5V renamed VBUS
- net VBUS: now also D4.1 (VDD), D5.1 (VDD), D6.1 (VDD)
- new net: D5.2 (DOUT), D6.4 (DIN)
- new net: D4.2 (DOUT), D5.4 (DIN)
- new net STATUS LIGHTS: D4.4 (DIN)
Other:
- note added: "Status Light's"
