File: Kicad/EDMX/EDMX.kicad_pcb (KiCad board)
At the start: 2 copper layers, 143 x 75.5 mm, 16 parts, among them J1 XLR3 IN, J2 Conn_01x04, J3 XLR3 OUT, M3 MountingHole_3.2mm_M3, Q1 2N3904, U1 MAX485E, U2 XIAO-ESP32-C3-DIP

Commit message: nano
Parts:
- added D4: DMX Status, LED_SMD:LED_WS2812B_PLCC4_5.0x5.0mm_P3.2mm, F.Cu at (154.5, 109.3)
- added D5: WiFi Status, LED_SMD:LED_WS2812B_PLCC4_5.0x5.0mm_P3.2mm, F.Cu at (146.6, 109.5)
- added D6: Light Control, LED_SMD:LED_WS2812B_PLCC4_5.0x5.0mm_P3.2mm, F.Cu at (138.6, 109.7)
- D1: footprint Diode_THT:D_DO-41_SOD81_P10.16mm_Horizontal -> Diode_THT:D_DO-34_SOD68_P10.16mm_Horizontal
- moved R4 7.62 mm to (149.5, 67.3), turned to 90 degrees
- moved R2 0.81 mm to (100.3, 66.0)
Connections:
- D1 pad 1: +5V -> VBUS
- D1 pad 2: Net-(D1-A) -> VBUS
- U1 pad 7: Net-(D2-A1) -> (no net)
- U1 pad 8: +5V -> VBUS
- U2 pad 14: Net-(D1-A) -> VBUS
- U2 pad 9: unconnected-(U2-GPIO8/D8/SCK-Pad9) -> STATUS LIGHTS
Routing:
- net GND: track 222.7 -> 2.55 mm
- net VBUS: track 0.00 -> 218.7 mm, vias 0 -> 1
- net +5V: track 150.7 -> 0.00 mm
- net TX: track 0.00 -> 78.6 mm
- net Net-(D1-A): track 13.5 -> 0.00 mm
- net STATUS LIGHTS: track 0.00 -> 12.5 mm
- added copper zone on B.Cu, net GND
- added copper zone on F.Cu, net GND
Other:
- board text added: "Endevour DMX"

Commit message: Updated Journal and moved the files about
Routing:
- net Net-(J1-Pad3): track 100.6 -> 98.7 mm
- removed copper zone on B.Cu, net GND
